Commit message: Footprint Joint changed to fixed

File: gazebo/gazebo.urdf.xacro (robot description, xacro)
@@ -3,7 +3,8 @@
 	<gazebo>
 		<plugin name="gazebo_ros_controller_manager" filename="libgazebo_ros_control.so">
+			<legacyModeNS>true</legacyModeNS>
 			<robotNamespace>/hyq2max</robotNamespace>
-			<robotSimType>dls_gazebo_interface/DLSHWSim</robotSimType>
-			<controlPeriod>0.004</controlPeriod>
+			<!--robotSimType>dls_gazebo_interface/DLSHWSim</robotSimType>
+			<controlPeriod>0.004</controlPeriod-->
 		</plugin>
 		<plugin filename="libgazebo_ros_p3d.so" name="gazebo_ros_p3d">

File: robots/hyq2max.urdf.xacro (robot description, xacro)
@@ -31,5 +31,5 @@
 	<!-- Trunk -->
 	<xacro:hyq2max_trunk name="base">
-		<origin xyz="-0.443 -0.191 -0.276" rpy="0 0 0"/>
+		<!--origin xyz="-0.443 -0.191 -0.276" rpy="0 0 0"/-->
 	</xacro:hyq2max_trunk>
 	<!-- LF leg -->

File: robots/hyq2max_model.urdf.xacro (robot description, xacro)
@@ -20,5 +20,5 @@
 	<!-- Trunk -->
 	<xacro:hyq2max_trunk name="base">
-		<origin xyz="-0.443 -0.191 -0.276" rpy="0 0 0"/>
+		<!--origin xyz="-0.443 -0.191 -0.276" rpy="0 0 0"/-->
 	</xacro:hyq2max_trunk>
 	<!-- LF leg -->

File: urdfs/leg/leg.transmission.xacro (robot description, xacro)
@@ -6,8 +6,8 @@
 			<type>transmission_interface/SimpleTransmission</type>
 			<joint name="${name}_haa_joint">
-				<hardwareInterface>EffortJointInterface</hardwareInterface>
+				<hardwareInterface>hardware_interface/EffortJointInterface</hardwareInterface>
 			</joint>
 			<actuator name="${name}_haa_motor">
-				<hardwareInterface>EffortJointInterface</hardwareInterface>
+				<hardwareInterface>hardware_interface/EffortJointInterface</hardwareInterface>
 				<mechanicalReduction>1</mechanicalReduction>
 			</actuator>
@@ -17,8 +17,8 @@
 			<type>transmission_interface/SimpleTransmission</type>
 			<joint name="${name}_hfe_joint">
-				<hardwareInterface>EffortJointInterface</hardwareInterface>
+				<hardwareInterface>hardware_interface/EffortJointInterface</hardwareInterface>
 			</joint>
 			<actuator name="${name}_hfe_motor">
-				<hardwareInterface>EffortJointInterface</hardwareInterface>
+				<hardwareInterface>hardware_interface/EffortJointInterface</hardwareInterface>
 				<mechanicalReduction>1</mechanicalReduction>
 			</actuator>
@@ -28,8 +28,8 @@
 			<type>transmission_interface/SimpleTransmission</type>
 			<joint name="${name}_kfe_joint">
-				<hardwareInterface>EffortJointInterface</hardwareInterface>
+				<hardwareInterface>hardware_interface/EffortJointInterface</hardwareInterface>
 			</joint>
 			<actuator name="${name}_kfe_motor">
-				<hardwareInterface>EffortJointInterface</hardwareInterface>
+				<hardwareInterface>hardware_interface/EffortJointInterface</hardwareInterface>
 				<mechanicalReduction>1</mechanicalReduction>
 			</actuator>

File: urdfs/trunk/trunk_model.urdf.xacro (robot description, xacro)
@@ -7,5 +7,5 @@
 	<xacro:macro name="hyq2max_trunk" params="name">
 		<!-- Floating-base Joint -->
-		<joint name="floating_base" type="floating">
+		<joint name="floating_base" type="fixed">
 			<origin xyz="0 0 0" rpy="0 0 0"/>
 			<parent link="${name}_link"/>

Commit message: Update rviz file and ground tf publisher

File: gazebo/gazebo.urdf.xacro (robot description, xacro)
@@ -18,4 +18,5 @@
 			<alwaysOn>true</alwaysOn>
 			<updateRate>250.0</updateRate>
+			<tf_prefix>tf</tf_prefix>
 		</plugin>
 	</gazebo>

File: robots/hyq2max_model.urdf.xacro (robot description, xacro)
@@ -28,5 +28,5 @@
 		reflect_left="1"
 		reflect_front="1"
-		load_force_sensors="false">
+		load_force_sensors="true">
 		<!-- <origin xyz="0.4435 0.097 0" rpy="${PI} ${PI/2} 0"/>  -->
 		<origin xyz="${haa_fh/2} ${haa_lr/2} 0" rpy="${PI} ${PI/2} 0"/>
@@ -38,5 +38,5 @@
 		reflect_left="-1"
 		reflect_front="1"
-		load_force_sensors="false">
+		load_force_sensors="true">
 		<!-- <origin xyz="0.4435 -0.097 0" rpy="0 ${PI/2} 0"/> -->
 		<origin xyz="${haa_fh/2} ${-haa_lr/2} 0" rpy="0 ${PI/2} 0"/>
@@ -48,5 +48,5 @@
 		reflect_left="1"
 		reflect_front="-1"
-		load_force_sensors="false">
+		load_force_sensors="true">
 		<!-- <origin xyz="-0.4435 0.097 0" rpy="${PI} ${PI/2} 0"/>  -->
 		<origin xyz="${-haa_fh/2} ${haa_lr/2} 0" rpy="${PI} ${PI/2} 0"/>
@@ -58,5 +58,5 @@
 		reflect_left="-1"
 		reflect_front="-1"
-		load_force_sensors="false">
+		load_force_sensors="true">
 		<!-- <origin xyz="-0.4435 -0.097 0" rpy="0 ${PI/2} 0"/> -->
 		<origin xyz="${-haa_fh/2} ${-haa_lr/2} 0" rpy="0 ${PI/2} 0"/>

File: urdfs/leg/leg.gazebo.xacro (robot description, xacro)
@@ -17,4 +17,5 @@
 		<gazebo reference="${name}_kfe_joint">
 			<provideFeedback>true</provideFeedback>
+			<preserveFixedJoint>true</preserveFixedJoint>
 		</gazebo>
 		<xacro:if value="${load_force_sensors}">
@@ -50,36 +51,53 @@
 			<minDepth>0.00</minDepth>
 		</gazebo>
-    	 <gazebo reference="${name}_lowerleg">
-            <kp>1000000.0</kp>
-            <kd>100.0</kd>
-            <mu1>1.5</mu1>
-            <mu2>1.5</mu2>
-            <fdir1>1 0 0</fdir1>
-            <maxVel>1.0</maxVel>
-            <minDepth>0.00</minDepth>
-            <sensor name="${name}_shin_contact_sensor" type="contact">
-                <always_on>true</always_on>
-                <update_rate>1000.0</update_rate>
-                <contact>
-                  <collision>${name}_lowerleg_collision</collision>
-                </contact>
-                <plugin name="${name}_shin_bumper" filename="libgazebo_ros_bumper.so">
-                  <bumperTopicName>/${name}_shin_sensor</bumperTopicName>
-                </plugin>
-            </sensor>
-        </gazebo>
+	    <gazebo reference="${name}_lowerleg">
+			<!--kp>1000000.0</kp>
+			<kd>100.0</kd>
+			<mu1>1.5</mu1>
+			<mu2>1.5</mu2>
+			<fdir1>1 0 0</fdir1>
+			<maxVel>1.0</maxVel>
+			<minDepth>0.00</minDepth-->
+			<mu1 value="50.0"/>
+            <mu2 value="50.0"/>
+            <kp value="10000000.0" />
+            <kd value="1.0" />
+            <minDepth value="0.005"/>
+			<sensor name="${name}_shin_contact_sensor" type="contact">
+				<always_on>true</always_on>
+				<update_rate>1000.0</update_rate>
+				<contact>
+					<!--collision>${name}_lowerleg_fixed_joint_lump__${name}_foot_collision_collision_1</collision-->
+					<!--collision>${name}_lowerleg_collision_collision</collision-->
+					<collision>${name}_lowerleg_collision_collision</collision>
+				</contact>
+				<plugin name="${name}_shin_bumper" filename="libgazebo_ros_bumper.so">
+					<bumperTopicName>/${name}_lowerleg_bumper</bumperTopicName>
+					<frameName>trunk</frameName>
+				</plugin>
+			</sensor>
+		</gazebo>
 		<gazebo reference="${name}_foot">
+			<mu1 value="50.0"/>
+            <mu2 value="50.0"/>
+            <kp value="10000000.0" />
+            <kd value="1.0" />
+            <minDepth value="0.005"/>
 			<sensor name="${name}_foot_contact_sensor" type="contact">
 				<always_on>true</always_on>
 				<update_rate>1000.0</update_rate>
 				<contact>
-					<collision>${name}_foot_collision</collision>
+					<!--collision>${name}_foot_collision</collision-->
+					<collision>${name}_lowerleg_fixed_joint_lump__${name}_foot_collision_collision_1</collision>
 				</contact>
 				<plugin name="${name}_foot_bumper" filename="libgazebo_ros_bumper.so">
-					<bumperTopicName>/${name}_grf</bumperTopicName>
-					<frameName>base_link</frameName>
+					<bumperTopicName>/${name}_foot_bumper</bumperTopicName>
+					<frameName>trunk</frameName>
 				</plugin>
 			</sensor>
 		</gazebo>
+		<gazebo reference="${name}_foot_joint">
+			<provideFeedback>true</provideFeedback>
+		</gazebo>
 	</xacro:macro>
 </robot>

File: urdfs/leg/leg.transmission.xacro (robot description, xacro)
@@ -35,4 +35,15 @@
 			</actuator>
 		</transmission>
+		<!-- Foot leg -->
+		<transmission name="${name}_kfe_trans">
+			<type>transmission_interface/SimpleTransmission</type>
+			<joint name="${name}_kfe_joint">
+				<hardwareInterface>hardware_interface/EffortJointInterface</hardwareInterface>
+			</joint>
+			<actuator name="${name}_kfe_motor">
+				<hardwareInterface>hardware_interface/EffortJointInterface</hardwareInterface>
+				<mechanicalReduction>1</mechanicalReduction>
+			</actuator>
+		</transmission>
 	</xacro:macro>
 </robot>

File: urdfs/leg/leg.urdf.xacro (robot description, xacro)
@@ -120,5 +120,6 @@
 				<material name="white"/>
 			</visual>
-			<collision>
+			<!--collision-->
+			<collision name="${name}_lowerleg_collision">
 				<origin xyz="0 0 0" rpy="${(1-reflect_front)*PI/2} 0 ${PI-reflect_front*knee_offset_angle*PI/180}"/>
 				<geometry>
@@ -141,5 +142,6 @@
                                 <material name="black"/>
 			</visual>
-			<collision>
+			<!--collision-->
+			<collision name="${name}_foot_collision">
 				<origin xyz="0 0 0" rpy="0 0 0"/>
 				<geometry>

File: urdfs/trunk/trunk_model.urdf.xacro (robot description, xacro)
@@ -7,12 +7,12 @@
 	<xacro:macro name="hyq2max_trunk" params="name">
 		<!-- Floating-base Joint -->
-		<joint name="floating_base" type="fixed">
+		<!--joint name="floating_base" type="fixed">
 			<origin xyz="0 0 0" rpy="0 0 0"/>
 			<parent link="${name}_link"/>
 			<child link="trunk"/>
-		</joint>
+		</joint-->
 		<!-- Links -->
 		<!-- Footprint link -->
-		<link name="${name}_link">
+		<!--link name="${name}_link">
 			<visual>
 				<geometry>
@@ -20,5 +20,5 @@
 				</geometry>
 			</visual>
-		</link>
+		</link-->
 		<!-- Trunk link -->
 		<link name="trunk">
